File: burger_king_light/burger_king_light.kicad_sch (KiCad schematic)
At the start: 3 parts, among them J1 Jack-DC

Commit message: resized mounting holes
Parts:
- H1, H2: footprint MountingHole:MountingHole_3.5mm_Pad_TopBottom -> MountingHole:MountingHole_2.5mm_Pad_TopBottom
Changed lines of the file:
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@@
 			)
 		)
-		(property "Footprint" "MountingHole:MountingHole_3.5mm_Pad_TopBottom"
+		(property "Footprint" "MountingHole:MountingHole_2.5mm_Pad_TopBottom"
 			(at 218.44 50.8 0)
 			(hide yes)
@@
 			)
 		)
-		(property "Footprint" "MountingHole:MountingHole_3.5mm_Pad_TopBottom"
+		(property "Footprint" "MountingHole:MountingHole_2.5mm_Pad_TopBottom"
 			(at 218.44 62.23 0)
 			(hide yes)
