File: burger_king_light/boost_converter.kicad_sch (KiCad schematic)
At the start: 1 part, among them IC1 TPS55340PWPR

Commit message: added all parts with references and purchase URLs
Parts:
- added Ccomp: 47nF, Capacitor_SMD:C_1206_3216Metric, symbol Device:C
- added Ccomp2: 820pF, Capacitor_SMD:C_0805_2012Metric, symbol Device:C
- added Cin: 10uF, Capacitor_SMD:C_1812_4532Metric, symbol Device:C
- added Cinx: 100nF, Capacitor_SMD:C_0805_2012Metric, symbol Device:C
- added Cout: EEHZA1H100R, EEHZA1H100R:CAP_EEHZA1H100R, symbol passives:EEHZA1H100R
- added Coutx: 2.2uF, Capacitor_SMD:C_0805_2012Metric, symbol Device:C
- added Css: 27nF, Capacitor_SMD:C_1206_3216Metric, symbol Device:C
- added D1: 550 mV @ 5 A, Diode_SMD:D_SMA, symbol Device:D_Zener_Filled
- added L1: IHLP2525CZER100M11, IND_IHLP_2525_CZ_VIS, symbol passives:IHLP2525CZER100M11
- added Rcomp: 2.55K, Resistor_SMD:R_1206_3216Metric, symbol Device:R_US
- added Rfbb: 10K, Resistor_SMD:R_1206_3216Metric, symbol Device:R_US
- added Rfbt: 249K, Resistor_SMD:R_1206_3216Metric, symbol Device:R_US
- added Rt: 47.5K, Resistor_SMD:R_1206_3216Metric, symbol Device:R_US
Other:
- moved on the sheet: IC1

Commit message: finished diagram
Parts:
- Cout: value EEHZA1H100R -> 10uF
Connections:
- net +32V: now reaches Cout.1
- net +32V: now also Coutx.1, D1.1 (K), Rfbt.1
- net GND: now reaches Cout.2
- net GND: now also Ccomp.2, Ccomp2.2, Cin.2, Cinx.2, Coutx.2, Css.2, IC1.11 (NC), IC1.12 (PGND_1), IC1.13 (PGND_2), IC1.14 (PGND_3), IC1.15 (EPAD), IC1.7 (AGND), Rfbb.2, Rt.1
- net at Ccomp.1: now also Rcomp.2
- net at Rfbt.2: now also IC1.9 (FB), Rfbb.1
- net at Rcomp.1: now also Ccomp2.1, IC1.8 (COMP)
- net at L1.1: now also D1.2 (A), IC1.1 (SW_1), IC1.2 (SW_2)
- net +12V: now reaches L1.2
- net +12V: now also Cin.1, Cinx.1, IC1.3 (VIN), IC1.4 (EN)
- net at Rt.2: now also IC1.10 (FREQ)
- net at Css.1: now also IC1.5 (SS)
- no-connect marks 0 -> 1
Other:
- moved on the sheet: Ccomp, Ccomp2, Cin, Cinx, Cout, Coutx, Css, D1, IC1, L1, Rcomp, Rfbb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

Commit message: excluded everything from simulation (temp fix)
Parts:
- renumbered Ccomp to Ccomp1, Cin to Cin1, Cinx to Cinx1, Cout to Cout1, Coutx to Coutx1, Css to Css1, Rcomp to Rcomp1, Rfbb to Rfbb1, Rfbt to Rfbt1, Rt to Rt1
Changed lines of the file:
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@@
 		(unit 1)
 		(body_style 1)
-		(exclude_from_sim no)
+		(exclude_from_sim yes)
 		(in_bom yes)
 		(on_board yes)
@@
 		(dnp no)
 		(fields_autoplaced yes)
-		(property "Reference" "Cout"
+		(property "Reference" "Cout1"
 			(at 213.36 107.3765 90)
 			(show_name no)
@@
 			(project "burger_king_light"
 				(path "/a1df17e6-efc5-454a-8f2a-f09b9061eebb/2b973585-e867-4f75-9aeb-d45cf169fa75"
-					(reference "Cout")
+					(reference "Cout1")
 					(unit 1)
 				)
@@
 		(unit 1)
 		(body_style 1)
-		(exclude_from_sim no)
+		(exclude_from_sim yes)
 		(in_bom yes)
 		(on_board yes)
@@
 		(unit 1)
 		(body_style 1)
-		(exclude_from_sim no)
+		(exclude_from_sim yes)
 		(in_bom yes)
 		(on_board yes)
@@
 		(dnp no)
 		(fields_autoplaced yes)
-		(property "Reference" "Ccomp"
+		(property "Reference" "Ccomp1"
 			(at 179.07 125.7299 0)
 			(show_name no)
@@
 			(project "burger_king_light"
 				(path "/a1df17e6-efc5-454a-8f2a-f09b9061eebb/2b973585-e867-4f75-9aeb-d45cf169fa75"
-					(reference "Ccomp")
+					(reference "Ccomp1")
 					(unit 1)
 				)
@@
 		(unit 1)
 		(body_style 1)
-		(exclude_from_sim no)
+		(exclude_from_sim yes)
 		(in_bom yes)
 		(on_board yes)
@@
 		(dnp no)
 		(fields_autoplaced yes)
-		(property "Reference" "Rfbt"
+		(property "Reference" "Rfbt1"
 			(at 199.39 101.5999 0)
 			(show_name no)
@@
 			(project "burger_king_light"
 				(path "/a1df17e6-efc5-454a-8f2a-f09b9061eebb/2b973585-e867-4f75-9aeb-d45cf169fa75"
-					(reference "Rfbt")
+					(reference "Rfbt1")
 					(unit 1)
 				)
@@
 		(unit 1)
 		(body_style 1)
-		(exclude_from_sim no)
+		(exclude_from_sim yes)
 		(in_bom yes)
 		(on_board yes)
@@
 		(dnp no)
 		(fields_autoplaced yes)
-		(property "Reference" "Rcomp"
+		(property "Reference" "Rcomp1"
 			(at 166.37 113.03 90)
 			(show_name no)
@@
 			(project "burger_king_light"
 				(path "/a1df17e6-efc5-454a-8f2a-f09b9061eebb/2b973585-e867-4f75-9aeb-d45cf169fa75"
-					(reference "Rcomp")
+					(reference "Rcomp1")
 					(unit 1)
 				)
@@
 		(unit 1)
 		(body_style 1)
-		(exclude_from_sim no)
+		(exclude_from_sim yes)
 		(in_bom yes)
 		(on_board yes)
@@
 		(unit 1)
 		(body_style 1)
-		(exclude_from_sim no)
+		(exclude_from_sim yes)
 		(in_bom yes)
 		(on_board yes)
@@
 		(unit 1)
 		(body_style 1)
-		(exclude_from_sim no)
+		(exclude_from_sim yes)
 		(in_bom yes)
 		(on_board yes)
@@
 		(dnp no)
 		(fields_autoplaced yes)
-		(property "Reference" "Rt"
+		(property "Reference" "Rt1"
 			(at 165.1 100.33 90)
 			(show_name no)
@@
 			(project "burger_king_light"
 				(path "/a1df17e6-efc5-454a-8f2a-f09b9061eebb/2b973585-e867-4f75-9aeb-d45cf169fa75"
-					(reference "Rt")
+					(reference "Rt1")
 					(unit 1)
 				)
@@
 		(unit 1)
 		(body_style 1)
-		(exclude_from_sim no)
+		(exclude_from_sim yes)
 		(in_bom yes)
 		(on_board yes)
@@
 		(dnp no)
 		(fields_autoplaced yes)
-		(property "Reference" "Rfbb"
+		(property "Reference" "Rfbb1"
 			(at 199.39 113.0299 0)
 			(show_name no)
@@
 			(project "burger_king_light"
 				(path "/a1df17e6-efc5-454a-8f2a-f09b9061eebb/2b973585-e867-4f75-9aeb-d45cf169fa75"
-					(reference "Rfbb")
+					(reference "Rfbb1")
 					(unit 1)
 				)
@@
 		(unit 1)
 		(body_style 1)
-		(exclude_from_sim no)
+		(exclude_from_sim yes)
 		(in_bom yes)
 		(on_board yes)
@@
 		(dnp no)
 		(fields_autoplaced yes)
-		(property "Reference" "Css"
+		(property "Reference" "Css1"
 			(at 111.76 119.3799 0)
 			(show_name no)
@@
 			(project "burger_king_light"
 				(path "/a1df17e6-efc5-454a-8f2a-f09b9061eebb/2b973585-e867-4f75-9aeb-d45cf169fa75"
-					(reference "Css")
+					(reference "Css1")
 					(unit 1)
 				)
@@
 		(unit 1)
 		(body_style 1)
-		(exclude_from_sim no)
+		(exclude_from_sim yes)
 		(in_bom yes)
 		(on_board yes)
@@
 		(dnp no)
 		(fields_autoplaced yes)
-		(property "Reference" "Cin"
+		(property "Reference" "Cin1"
 			(at 86.36 107.9499 0)
 			(show_name no)
@@
 			(project "burger_king_light"
 				(path "/a1df17e6-efc5-454a-8f2a-f09b9061eebb/2b973585-e867-4f75-9aeb-d45cf169fa75"
-					(reference "Cin")
+					(reference "Cin1")
 					(unit 1)
 				)
@@
 		(unit 1)
 		(body_style 1)
-		(exclude_from_sim no)
+		(exclude_from_sim yes)
 		(in_bom yes)
 		(on_board yes)
@@
 		(unit 1)
 		(body_style 1)
-		(exclude_from_sim no)
+		(exclude_from_sim yes)
 		(in_bom yes)
 		(on_board yes)
@@
 		(dnp no)
 		(fields_autoplaced yes)
-		(property "Reference" "Coutx"
+		(property "Reference" "Coutx1"
 			(at 226.06 107.9499 0)
 			(show_name no)
@@
 			(project "burger_king_light"
 				(path "/a1df17e6-efc5-454a-8f2a-f09b9061eebb/2b973585-e867-4f75-9aeb-d45cf169fa75"
-					(reference "Coutx")
+					(reference "Coutx1")
 					(unit 1)
 				)
@@
 		(unit 1)
 		(body_style 1)
-		(exclude_from_sim no)
+		(exclude_from_sim yes)
 		(in_bom yes)
 		(on_board yes)
@@
 		(unit 1)
 		(body_style 1)
-		(exclude_from_sim no)
+		(exclude_from_sim yes)
 		(in_bom yes)
 		(on_board yes)
@@
 		(unit 1)
 		(body_style 1)
-		(exclude_from_sim no)
+		(exclude_from_sim yes)
 		(in_bom yes)
 		(on_board yes)
@@
 		(unit 1)
 		(body_style 1)
-		(exclude_from_sim no)
+		(exclude_from_sim yes)
 		(in_bom yes)
 		(on_board yes)
@@
 		(unit 1)
 		(body_style 1)
-		(exclude_from_sim no)
+		(exclude_from_sim yes)
 		(in_bom yes)
 		(on_board yes)
@@
 		(dnp no)
 		(fields_autoplaced yes)
-		(property "Reference" "Cinx"
+		(property "Reference" "Cinx1"
 			(at 99.06 107.9499 0)
 			(show_name no)
@@
 			(project "burger_king_light"
 				(path "/a1df17e6-efc5-454a-8f2a-f09b9061eebb/2b973585-e867-4f75-9aeb-d45cf169fa75"
-					(reference "Cinx")
-					(unit 1)
-				)
+					(reference "Cinx1")
+					(unit 1)
+				)
