File: burger_king_light/astable_555.kicad_sch (KiCad schematic)
At the start: 14 parts, among them U1 ICM7555CBAZ

Commit message: changed IC reference designators to U
Parts:
- RV1: footprint (none) -> passives:3-PIN POT
- renumbered U1 to U2
Changed lines of the file:
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@@
 		(in_pos_files yes)
 		(dnp no)
-		(property "Reference" "U1"
+		(property "Reference" "U2"
 			(at 184.404 81.026 0)
 			(show_name no)
@@
 			(project "burger_king_light"
 				(path "/a1df17e6-efc5-454a-8f2a-f09b9061eebb/0641335a-b39f-4dc9-bc4d-328a71cdee24"
-					(reference "U1")
+					(reference "U2")
 					(unit 1)
 				)
@@
 			)
 		)
-		(property "Footprint" ""
+		(property "Footprint" "passives:3-PIN POT"
 			(at 200.66 100.33 0)
 			(hide yes)
