File: burger_king_light/led_drivers.kicad_sch (KiCad schematic)
At the start: 18 parts, among them IC2 IS32LT3178-GRLA3-TR, IC3 IS32LT3178-GRLA3-TR, IC4 IS32LT3178-GRLA3-TR

Commit message: changed IC reference designators to U
Parts:
- renumbered IC2 to U3, IC3 to U4, IC4 to U5
Changed lines of the file:
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@@
 		(dnp no)
 		(fields_autoplaced yes)
-		(property "Reference" "IC4"
+		(property "Reference" "U5"
 			(at 106.68 124.46 0)
 			(show_name no)
@@
 			(project "burger_king_light"
 				(path "/a1df17e6-efc5-454a-8f2a-f09b9061eebb/8d1794ed-4131-430d-a90f-cb9174cf4871"
-					(reference "IC4")
+					(reference "U5")
 					(unit 1)
 				)
@@
 		(dnp no)
 		(fields_autoplaced yes)
-		(property "Reference" "IC2"
+		(property "Reference" "U3"
 			(at 106.68 17.78 0)
 			(show_name no)
@@
 			(project "burger_king_light"
 				(path "/a1df17e6-efc5-454a-8f2a-f09b9061eebb/8d1794ed-4131-430d-a90f-cb9174cf4871"
-					(reference "IC2")
+					(reference "U3")
 					(unit 1)
 				)
@@
 		(dnp no)
 		(fields_autoplaced yes)
-		(property "Reference" "IC3"
+		(property "Reference" "U4"
 			(at 106.68 72.39 0)
 			(show_name no)
@@
 			(project "burger_king_light"
 				(path "/a1df17e6-efc5-454a-8f2a-f09b9061eebb/8d1794ed-4131-430d-a90f-cb9174cf4871"
-					(reference "IC3")
+					(reference "U4")
 					(unit 1)
 				)
