File: burger_king_light/led_drivers.kicad_sch (KiCad schematic)
At the start: 18 parts, among them U3 IS32LT3178-GRLA3-TR, U4 IS32LT3178-GRLA3-TR, U5 IS32LT3178-GRLA3-TR

Commit message: resized mounting holes
Parts:
- H3, H4, H5, H6, H7, H8: footprint MountingHole:MountingHole_3.5mm_Pad_TopBottom -> MountingHole:MountingHole_2.5mm_Pad_TopBottom
Changed lines of the file:
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@@
 			)
 		)
-		(property "Footprint" "MountingHole:MountingHole_3.5mm_Pad_TopBottom"
+		(property "Footprint" "MountingHole:MountingHole_2.5mm_Pad_TopBottom"
 			(at 184.15 36.83 0)
 			(hide yes)
@@
 			)
 		)
-		(property "Footprint" "MountingHole:MountingHole_3.5mm_Pad_TopBottom"
+		(property "Footprint" "MountingHole:MountingHole_2.5mm_Pad_TopBottom"
 			(at 184.15 143.51 0)
 			(hide yes)
@@
 			)
 		)
-		(property "Footprint" "MountingHole:MountingHole_3.5mm_Pad_TopBottom"
+		(property "Footprint" "MountingHole:MountingHole_2.5mm_Pad_TopBottom"
 			(at 184.15 48.26 0)
 			(hide yes)
@@
 			)
 		)
-		(property "Footprint" "MountingHole:MountingHole_3.5mm_Pad_TopBottom"
+		(property "Footprint" "MountingHole:MountingHole_2.5mm_Pad_TopBottom"
 			(at 184.15 154.94 0)
 			(hide yes)
@@
 			)
 		)
-		(property "Footprint" "MountingHole:MountingHole_3.5mm_Pad_TopBottom"
+		(property "Footprint" "MountingHole:MountingHole_2.5mm_Pad_TopBottom"
 			(at 184.15 91.44 0)
 			(hide yes)
@@
 			)
 		)
-		(property "Footprint" "MountingHole:MountingHole_3.5mm_Pad_TopBottom"
+		(property "Footprint" "MountingHole:MountingHole_2.5mm_Pad_TopBottom"
 			(at 184.15 102.87 0)
 			(hide yes)
