File: burger_king_light/burger_king_light.kicad_pcb (KiCad board)
At the start: 4 copper layers, 102.1 x 58.7 mm, 57 parts, among them U1 TPS55340PWPR, U2 ICM7555CBAZ, U3 IS32LT3178-GRLA3-TR, U4 IS32LT3178-GRLA3-TR, U5 IS32LT3178-GRLA3-TR

Commit message: resized 555 IC secion, changed pot footprint
Parts:
- H1, H2, H3, H4, H5, H6, H7, H8: footprint MountingHole:MountingHole_3.5mm_Pad_TopBottom -> MountingHole:MountingHole_2.5mm_Pad_TopBottom
- moved RV1 13.1 mm to (86.0, 124.0)
- moved D4 9.77 mm to (93.0, 116.3), turned to 90 degrees
- moved D3 9.06 mm to (99.1, 116.3), turned to -90 degrees
Routing:
- net Net-(D4-K): track 11.5 -> 4.20 mm
- net Net-(R3-Pad2): track 23.6 -> 19.2 mm
- net Net-(D2-K): track 22.1 -> 18.0 mm
- net PWM out: track 133.1 -> 129.2 mm
- net Net-(D3-A): track 6.98 -> 4.36 mm
- net 0: vias 166 -> 169
